File: Hardware/System/backpackbuddy_system/power.kicad_sch (KiCad schematic)
At the start: 34 parts, among them J11 Battery, Q3 SIHF9Z24STRR-GE3, U2 SI-8050Y, U3 LM3940

Commit message: schematic mostly done, just need to fix ERC, decoup caps, TP
Parts:
- added JP1: SolderJumper_2_Open, Jumper:SolderJumper-2_P1.3mm_Open_RoundedPad1.0x1.5mm, symbol Jumper:SolderJumper_2_Open
Connections:
- net +9V: now also JP1.2 (B)
- net at F2.1, J11.2 (Pin_2): now also JP1.1 (A)
Other:
- moved on the sheet: C10, C11, C12, C13, C6, C7, C8, C9, D2, D3, D4, D5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

Commit message: random other sch changes
Parts:
- J11: footprint Connector_Molex:Molex_KK-254_AE-6410-03A_1x03_P2.54mm_Vertical -> Connector_PinHeader_2.54mm:PinHeader_1x03_P2.54mm_Vertical; MPN 0022232031 -> (none); Stock https://www.digikey.com/en/products/detail/molex/0022232031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 -> In connector kit
- JP1: value SolderJumper_2_Open -> PP Short
- TP1: Note 9V Power -> 18V Power
- TP3: Note Protected 9V -> Protected 18V
Connections:
- net +9V renamed 18V PROTECTED
Other:
- note removed: "9V PROTECTED"
Changed lines of the file:
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@@
   (junction (at 116.84 173.99) (diameter 0) (color 0 0 0 0)
   )
-  (junction (at 158.75 48.26) (diameter 0) (color 0 0 0 0)
-  )
   (junction (at 135.89 48.26) (diameter 0) (color 0 0 0 0)
   )
@@
     (stroke (width 0) (type default) (color 0 0 0 0))
   )
-  (wire (pts (xy 152.4 48.26) (xy 158.75 48.26))
+  (wire (pts (xy 152.4 48.26) (xy 171.45 48.26))
     (stroke (width 0) (type default) (color 0 0 0 0))
   )
@@
     (stroke (width 0) (type default) (color 0 0 0 0))
   )
+  (wire (pts (xy 152.4 33.02) (xy 127 33.02))
+    (stroke (width 0) (type default) (color 0 0 0 0))
+  )
   (wire (pts (xy 59.69 147.32) (xy 59.69 173.99))
     (stroke (width 0) (type default) (color 0 0 0 0))
@@
     (stroke (width 0) (type default) (color 0 0 0 0))
   )
-  (wire (pts (xy 158.75 33.02) (xy 158.75 48.26))
-    (stroke (width 0) (type default) (color 0 0 0 0))
-  )
-  (wire (pts (xy 40.64 130.81) (xy 40.64 128.27))
-    (stroke (width 0) (type default) (color 0 0 0 0))
-  )
   (wire (pts (xy 96.52 97.79) (xy 96.52 100.33))
     (stroke (width 0) (type default) (color 0 0 0 0))
@@
     (stroke (width 0) (type default) (color 0 0 0 0))
   )
-  (wire (pts (xy 127 33.02) (xy 158.75 33.02))
-    (stroke (width 0) (type default) (color 0 0 0 0))
-  )
   (wire (pts (xy 82.55 45.72) (xy 82.55 48.26))
     (stroke (width 0) (type default) (color 0 0 0 0))
@@
     (stroke (width 0) (type default) (color 0 0 0 0))
   )
+  (wire (pts (xy 171.45 48.26) (xy 171.45 46.99))
+    (stroke (width 0) (type default) (color 0 0 0 0))
+  )
   (wire (pts (xy 144.78 58.42) (xy 144.78 60.96))
     (stroke (width 0) (type default) (color 0 0 0 0))
   )
-  (wire (pts (xy 158.75 48.26) (xy 162.56 48.26))
-    (stroke (width 0) (type default) (color 0 0 0 0))
-  )
   (wire (pts (xy 149.86 139.7) (xy 156.21 139.7))
     (stroke (width 0) (type default) (color 0 0 0 0))
@@
     (stroke (width 0) (type default) (color 0 0 0 0))
   )
-  (wire (pts (xy 162.56 48.26) (xy 162.56 44.45))
-    (stroke (width 0) (type default) (color 0 0 0 0))
-  )
   (wire (pts (xy 115.57 48.26) (xy 115.57 50.8))
     (stroke (width 0) (type default) (color 0 0 0 0))
@@
     (stroke (width 0) (type default) (color 0 0 0 0))
   )
-  (wire (pts (xy 152.4 46.99) (xy 152.4 48.26))
+  (wire (pts (xy 152.4 33.02) (xy 152.4 48.26))
     (stroke (width 0) (type default) (color 0 0 0 0))
   )
@@
     (effects (font (size 3 3)) (justify left bottom))
   )
-  (text "9V PROTECTED" (at 128.27 48.26 0)
-    (effects (font (size 1.27 1.27)) (justify left bottom))
-  )
   (text "3.3V Regulator" (at 215.9 76.2 0)
     (effects (font (size 3 3)) (justify left bottom))
   )
+  (label "18V PROTECTED" (at 40.64 130.81 0)
+    (effects (font (size 1.27 1.27)) (justify left bottom))
+  )
+  (label "18V PROTECTED" (at 152.4 48.26 0)
+    (effects (font (size 1.27 1.27)) (justify left bottom))
+  )
   (hierarchical_label "+3V3" (shape output) (at 264.16 44.45 0)
     (effects (font (size 1.27 1.27)) (justify left))
@@
       (effects (font (size 1.27 1.27)) (justify left))
     )
-    (property "Footprint" "Connector_Molex:Molex_KK-254_AE-6410-03A_1x03_P2.54mm_Vertical" (id 2) (at 35.56 48.26 0)
+    (property "Footprint" "Connector_PinHeader_2.54mm:PinHeader_1x03_P2.54mm_Vertical" (id 2) (at 35.56 48.26 0)
       (effects (font (size 1.27 1.27)) hide)
     )
@@
       (effects (font (size 1.27 1.27)) hide)
     )
-    (property "MPN" "0022232031" (id 5) (at 35.56 48.26 0)
-      (effects (font (size 1.27 1.27)) hide)
-    )
-    (property "Stock" "https://www.digikey.com/en/products/detail/molex/0022232031/26669" (id 6) (at 35.56 48.26 0)
+    (property "MPN" "" (id 5) (at 35.56 48.26 0)
+      (effects (font (size 1.27 1.27)) hide)
+    )
+    (property "Stock" "In connector kit" (id 6) (at 35.56 48.26 0)
       (effects (font (size 1.27 1.27)) hide)
     )
@@
     (pin "1")
   )
-  (symbol (lib_id "power:+9V") (at 40.64 128.27 0) (unit 1)
-    (in_bom yes) (on_board yes)
-    (property "Reference" "#PWR028" (id 0) (at 40.64 132.08 0)
-      (effects (font (size 1.27 1.27)) hide)
-    )
-    (property "Value" "+9V" (id 1) (at 40.64 124.46 0))
-    (property "Footprint" "" (id 2) (at 40.64 128.27 0)
-      (effects (font (size 1.27 1.27)) hide)
-    )
-    (property "Datasheet" "" (id 3) (at 40.64 128.27 0)
-      (effects (font (size 1.27 1.27)) hide)
-    )
-    (pin "1")
-  )
   (symbol (lib_id "Connector:TestPoint") (at 149.86 138.43 0) (unit 1)
     (in_bom yes) (on_board yes) (fields_autoplaced)
@@
       (effects (font (size 1.27 1.27)) hide)
     )
-    (property "Note" "9V Power" (id 4) (at 82.55 36.83 0))
+    (property "Note" "18V Power" (id 4) (at 82.55 36.83 0))
     (property "DNP" "" (id 5) (at 82.55 45.72 0)
       (effects (font (size 1.27 1.27)) hide)
@@
     (pin "2")
   )
-  (symbol (lib_id "power:PWR_FLAG") (at 152.4 46.99 0) (unit 1)
-    (in_bom yes) (on_board yes)
-    (property "Reference" "#FLG02" (id 0) (at 152.4 45.085 0)
-      (effects (font (size 1.27 1.27)) hide)
-    )
-    (property "Value" "PWR_FLAG" (id 1) (at 152.4 42.5958 0))
-    (property "Footprint" "" (id 2) (at 152.4 46.99 0)
-      (effects (font (size 1.27 1.27)) hide)
-    )
-    (property "Datasheet" "~" (id 3) (at 152.4 46.99 0)
+  (symbol (lib_id "power:PWR_FLAG") (at 171.45 46.99 0) (unit 1)
+    (in_bom yes) (on_board yes)
+    (property "Reference" "#FLG02" (id 0) (at 171.45 45.085 0)
+      (effects (font (size 1.27 1.27)) hide)
+    )
+    (property "Value" "PWR_FLAG" (id 1) (at 171.45 42.5958 0))
+    (property "Footprint" "" (id 2) (at 171.45 46.99 0)
+      (effects (font (size 1.27 1.27)) hide)
+    )
+    (property "Datasheet" "~" (id 3) (at 171.45 46.99 0)
       (effects (font (size 1.27 1.27)) hide)
     )
@@
     (in_bom yes) (on_board yes) (fields_autoplaced)
     (property "Reference" "JP1" (id 0) (at 123.19 26.67 0))
-    (property "Value" "SolderJumper_2_Open" (id 1) (at 123.19 29.21 0))
+    (property "Value" "PP Short" (id 1) (at 123.19 29.21 0))
     (property "Footprint" "Jumper:SolderJumper-2_P1.3mm_Open_RoundedPad1.0x1.5mm" (id 2) (at 123.19 33.02 0)
       (effects (font (size 1.27 1.27)) hide)
@@
     (pin "1")
     (pin "2")
-  )
-  (symbol (lib_id "power:+9V") (at 162.56 44.45 0) (unit 1)
-    (in_bom yes) (on_board yes)
-    (property "Reference" "#PWR036" (id 0) (at 162.56 48.26 0)
-      (effects (font (size 1.27 1.27)) hide)
-    )
-    (property "Value" "+9V" (id 1) (at 162.56 40.64 0))
-    (property "Footprint" "" (id 2) (at 162.56 44.45 0)
-      (effects (font (size 1.27 1.27)) hide)
-    )
-    (property "Datasheet" "" (id 3) (at 162.56 44.45 0)
-      (effects (font (size 1.27 1.27)) hide)
-    )
-    (pin "1")
   )
   (symbol (lib_id "Device:C_Polarized") (at 46.99 143.51 0) (unit 1)
@@
       (effects (font (size 1.27 1.27)) hide)
     )
-    (property "Note" "Protected 9V" (id 4) (at 146.05 38.1 0))
+    (property "Note" "Protected 18V" (id 4) (at 143.51 38.1 0))
     (property "DNP" "" (id 5) (at 146.05 45.72 0)
       (effects (font (size 1.27 1.27)) hide)

Commit message: fixed an error
Changed lines of the file:
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@@
   (junction (at 96.52 97.79) (diameter 0) (color 0 0 0 0)
   )
-  (junction (at 218.44 58.42) (diameter 0) (color 0 0 0 0)
-  )
   (junction (at 82.55 48.26) (diameter 0) (color 0 0 0 0)
   )
@@
   (junction (at 52.07 48.26) (diameter 0) (color 0 0 0 0)
   )
-  (junction (at 59.69 48.26) (diameter 0) (color 0 0 0 0)
-  )
   (junction (at 147.32 139.7) (diameter 0) (color 0 0 0 0)
   )
@@
     (stroke (width 0) (type default) (color 0 0 0 0))
   )
-  (wire (pts (xy 218.44 58.42) (xy 218.44 60.96))
-    (stroke (width 0) (type default) (color 0 0 0 0))
-  )
   (wire (pts (xy 256.54 54.61) (xy 256.54 57.15))
     (stroke (width 0) (type default) (color 0 0 0 0))
@@
     (stroke (width 0) (type default) (color 0 0 0 0))
   )
-  (wire (pts (xy 218.44 58.42) (xy 227.33 58.42))
-    (stroke (width 0) (type default) (color 0 0 0 0))
-  )
   (wire (pts (xy 52.07 33.02) (xy 52.07 48.26))
     (stroke (width 0) (type default) (color 0 0 0 0))
@@
     (stroke (width 0) (type default) (color 0 0 0 0))
   )
-  (wire (pts (xy 59.69 48.26) (xy 64.77 48.26))
-    (stroke (width 0) (type default) (color 0 0 0 0))
-  )
   (wire (pts (xy 147.32 149.86) (xy 147.32 152.4))
     (stroke (width 0) (type default) (color 0 0 0 0))
@@
     (stroke (width 0) (type default) (color 0 0 0 0))
   )
-  (wire (pts (xy 212.09 58.42) (xy 218.44 58.42))
+  (wire (pts (xy 212.09 58.42) (xy 227.33 58.42))
     (stroke (width 0) (type default) (color 0 0 0 0))
   )
@@
     (stroke (width 0) (type default) (color 0 0 0 0))
   )
-  (wire (pts (xy 52.07 48.26) (xy 59.69 48.26))
+  (wire (pts (xy 52.07 48.26) (xy 64.77 48.26))
     (stroke (width 0) (type default) (color 0 0 0 0))
   )
@@
   )
   (wire (pts (xy 237.49 44.45) (xy 241.3 44.45))
-    (stroke (width 0) (type default) (color 0 0 0 0))
-  )
-  (wire (pts (xy 59.69 44.45) (xy 59.69 48.26))
     (stroke (width 0) (type default) (color 0 0 0 0))
   )
@@
     (pin "2")
   )
-  (symbol (lib_id "power:PWR_FLAG") (at 59.69 44.45 0) (unit 1)
-    (in_bom yes) (on_board yes)
-    (property "Reference" "#FLG01" (id 0) (at 59.69 42.545 0)
-      (effects (font (size 1.27 1.27)) hide)
-    )
-    (property "Value" "PWR_FLAG" (id 1) (at 59.69 40.0558 0))
-    (property "Footprint" "" (id 2) (at 59.69 44.45 0)
-      (effects (font (size 1.27 1.27)) hide)
-    )
-    (property "Datasheet" "~" (id 3) (at 59.69 44.45 0)
-      (effects (font (size 1.27 1.27)) hide)
-    )
-    (pin "1")
-  )
   (symbol (lib_id "Device:LED") (at 144.78 64.77 90) (unit 1)
     (in_bom yes) (on_board yes) (fields_autoplaced)
@@
       (effects (font (size 1.27 1.27)) hide)
     )
-    (pin "1")
-  )
-  (symbol (lib_id "power:PWR_FLAG") (at 218.44 60.96 180) (unit 1)
-    (in_bom yes) (on_board yes)
-    (property "Reference" "#FLG04" (id 0) (at 218.44 62.865 0)
-      (effects (font (size 1.27 1.27)) hide)
-    )
-    (property "Value" "PWR_FLAG" (id 1) (at 218.44 65.3542 0))
-    (property "Footprint" "" (id 2) (at 218.44 60.96 0)
-      (effects (font (size 1.27 1.27)) hide)
-    )
-    (property "Datasheet" "~" (id 3) (at 218.44 60.96 0)
-      (effects (font (size 1.27 1.27)) hide)
-    )

Commit message: fixed layout errors
Parts:
- C10, C11, C12, C14: footprint Capacitor_SMD:C_0603_1608Metric_Pad1.05x0.95mm_HandSolder -> Capacitor_SMD:C_0603_1608Metric_Pad1.08x0.95mm_HandSolder
- R4, R5, R6, R7, R8, R9: footprint Resistor_SMD:R_0603_1608Metric_Pad1.05x0.95mm_HandSolder -> Resistor_SMD:R_0603_1608Metric_Pad0.98x0.95mm_HandSolder
Changed lines of the file:
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@@
       (effects (font (size 1.27 1.27)) (justify left))
     )
-    (property "Footprint" "Capacitor_SMD:C_0603_1608Metric_Pad1.05x0.95mm_HandSolder" (id 2) (at 213.0552 55.88 0)
+    (property "Footprint" "Capacitor_SMD:C_0603_1608Metric_Pad1.08x0.95mm_HandSolder" (id 2) (at 213.0552 55.88 0)
       (effects (font (size 1.27 1.27)) hide)
     )
@@
       (effects (font (size 1.27 1.27)) (justify left))
     )
-    (property "Footprint" "Resistor_SMD:R_0603_1608Metric_Pad1.05x0.95mm_HandSolder" (id 2) (at 106.172 67.31 90)
+    (property "Footprint" "Resistor_SMD:R_0603_1608Metric_Pad0.98x0.95mm_HandSolder" (id 2) (at 106.172 67.31 90)
       (effects (font (size 1.27 1.27)) hide)
     )
@@
       (effects (font (size 1.27 1.27)) (justify left))
     )
-    (property "Footprint" "Resistor_SMD:R_0603_1608Metric_Pad1.05x0.95mm_HandSolder" (id 2) (at 143.002 54.61 90)
+    (property "Footprint" "Resistor_SMD:R_0603_1608Metric_Pad0.98x0.95mm_HandSolder" (id 2) (at 143.002 54.61 90)
       (effects (font (size 1.27 1.27)) hide)
     )
@@
       (effects (font (size 1.27 1.27)) (justify left))
     )
-    (property "Footprint" "Resistor_SMD:R_0603_1608Metric_Pad1.05x0.95mm_HandSolder" (id 2) (at 254.762 50.8 90)
+    (property "Footprint" "Resistor_SMD:R_0603_1608Metric_Pad0.98x0.95mm_HandSolder" (id 2) (at 254.762 50.8 90)
       (effects (font (size 1.27 1.27)) hide)
     )
@@
       (effects (font (size 1.27 1.27)) (justify left))
     )
-    (property "Footprint" "Resistor_SMD:R_0603_1608Metric_Pad1.05x0.95mm_HandSolder" (id 2) (at 145.542 146.05 90)
+    (property "Footprint" "Resistor_SMD:R_0603_1608Metric_Pad0.98x0.95mm_HandSolder" (id 2) (at 145.542 146.05 90)
       (effects (font (size 1.27 1.27)) hide)
     )
@@
       (effects (font (size 1.27 1.27)) (justify left))
     )
-    (property "Footprint" "Capacitor_SMD:C_0603_1608Metric_Pad1.05x0.95mm_HandSolder" (id 2) (at 116.5352 137.16 0)
+    (property "Footprint" "Capacitor_SMD:C_0603_1608Metric_Pad1.08x0.95mm_HandSolder" (id 2) (at 116.5352 137.16 0)
       (effects (font (size 1.27 1.27)) hide)
     )
@@
       (effects (font (size 1.27 1.27)) (justify left))
     )
-    (property "Footprint" "Resistor_SMD:R_0603_1608Metric_Pad1.05x0.95mm_HandSolder" (id 2) (at 134.112 90.17 90)
+    (property "Footprint" "Resistor_SMD:R_0603_1608Metric_Pad0.98x0.95mm_HandSolder" (id 2) (at 134.112 90.17 90)
       (effects (font (size 1.27 1.27)) hide)
     )
@@
       (effects (font (size 1.27 1.27)) (justify left))
     )
-    (property "Footprint" "Resistor_SMD:R_0603_1608Metric_Pad1.05x0.95mm_HandSolder" (id 2) (at 92.202 167.64 90)
+    (property "Footprint" "Resistor_SMD:R_0603_1608Metric_Pad0.98x0.95mm_HandSolder" (id 2) (at 92.202 167.64 90)
       (effects (font (size 1.27 1.27)) hide)
     )
@@
       (effects (font (size 1.27 1.27)) (justify left))
     )
-    (property "Footprint" "Capacitor_SMD:C_0603_1608Metric_Pad1.05x0.95mm_HandSolder" (id 2) (at 94.9452 160.02 0)
+    (property "Footprint" "Capacitor_SMD:C_0603_1608Metric_Pad1.08x0.95mm_HandSolder" (id 2) (at 94.9452 160.02 0)
       (effects (font (size 1.27 1.27)) hide)
     )
@@
       (effects (font (size 1.27 1.27)) (justify left))
     )
-    (property "Footprint" "Capacitor_SMD:C_0603_1608Metric_Pad1.05x0.95mm_HandSolder" (id 2) (at 116.5352 93.98 0)
-      (effects (font (size 1.27 1.27)) hide)
-    )
+    (property "Footprint" "Capacitor_SMD:C_0603_1608Metric_Pad1.08x0.95mm_HandSolder" (id 2) (at 116.5352 93.98 0)
+      (effects (font (size 1.27 1.27)) hide)
+    )

Commit message: fixed lm3940 symbol, changed crystal stuff
Parts:
- U3: MPN LM3940 -> (none); Stock Ordered! -> (none)
Connections:
- net GND: now also U3.4 (GND)
Changed lines of the file:
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@@
       (effects (font (size 1.27 1.27)) hide)
     )
-    (property "Datasheet" "~" (id 3) (at 116.84 154.94 0)
+    (property "Datasheet" "https://www.semicon.sanken-ele.co.jp/sk_content/fmw-2156_ds_en.pdf" (id 3) (at 116.84 154.94 0)
       (effects (font (size 1.27 1.27)) hide)
     )
@@
     )
     (pin "1")
-  )
-  (symbol (lib_id "Backpack_buddy_libraries:LM3940") (at 227.33 40.64 0) (unit 1)
-    (in_bom yes) (on_board yes) (fields_autoplaced)
-    (property "Reference" "U3" (id 0) (at 227.33 36.83 0))
-    (property "Value" "LM3940" (id 1) (at 227.33 39.37 0))
-    (property "Footprint" "Package_TO_SOT_SMD:SOT-223" (id 2) (at 227.33 38.1 0)
-      (effects (font (size 1.27 1.27)) hide)
-    )
-    (property "Datasheet" "https://www.ti.com/lit/ds/symlink/lm3940.pdf?HQS=dis-dk-null-digikeymode-dsf-pf-null-wwe&ts=1676759070206&ref_url=https%253A%252F%252Fwww.ti.com%252Fgeneral%252Fdocs%252Fsuppproductinfo.tsp%253FdistId%253D10%2526gotoUrl%253Dhttps%253A%252F%252Fwww.ti.com%252Flit%252Fgpn%252Flm3940" (id 3) (at 227.33 53.34 0)
-      (effects (font (size 1.27 1.27)) hide)
-    )
-    (property "MPN" "LM3940" (id 4) (at 227.33 40.64 0)
-      (effects (font (size 1.27 1.27)) hide)
-    )
-    (property "Stock" "Ordered!" (id 5) (at 227.33 40.64 0)
-      (effects (font (size 1.27 1.27)) hide)
-    )
-    (pin "1")
-    (pin "2")
-    (pin "3")
   )
   (symbol (lib_id "Connector:TestPoint") (at 259.08 41.91 0) (unit 1)
@@
     (pin "2")
   )
+  (symbol (lib_name "LM3940_1") (lib_id "Backpack_buddy_libraries:LM3940") (at 227.33 40.64 0) (unit 1)
+    (in_bom yes) (on_board yes) (fields_autoplaced)
+    (property "Reference" "U3" (id 0) (at 227.33 36.83 0))
+    (property "Value" "LM3940" (id 1) (at 227.33 39.37 0))
+    (property "Footprint" "Package_TO_SOT_SMD:SOT-223" (id 2) (at 227.33 38.1 0)
+      (effects (font (size 1.27 1.27)) hide)
+    )
+    (property "Datasheet" "https://www.ti.com/lit/ds/symlink/lm3940.pdf?HQS=dis-dk-null-digikeymode-dsf-pf-null-wwe&ts=1676759070206&ref_url=https%253A%252F%252Fwww.ti.com%252Fgeneral%252Fdocs%252Fsuppproductinfo.tsp%253FdistId%253D10%2526gotoUrl%253Dhttps%253A%252F%252Fwww.ti.com%252Flit%252Fgpn%252Flm3940" (id 3) (at 227.33 64.77 0)
+      (effects (font (size 1.27 1.27)) hide)
+    )
+    (pin "1")
+    (pin "2")
+    (pin "3")
+    (pin "4")
+  )
   (symbol (lib_id "Device:C_Polarized") (at 133.35 154.94 0) (unit 1)

Commit message: fixed table values
Parts:
- C11: Stock https://www.digikey.com/en/products/detail/kemet/C0603C104K5RAC7867/1465623?utm_adgroup=Ceramic%20Capacitors&utm_source=google&utm_medium=cpc&utm_campaign=Shopping_Product_Capacitors_NEW&utm_term=&utm_content=Ceramic%20Capacitors -> https://www.digikey.com/en/products/detail/kemet/C0603C104K5RAC3190/12701955?utm_adgroup=Capacitors&utm_source=google&utm_medium=cpc&utm_campaign=Shopping_Supplier_KEMET&utm_term=&utm_content=Capacitors
Changed lines of the file:
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@@
       (effects (font (size 1.27 1.27)) hide)
     )
-    (property "Stock" "https://www.digikey.com/en/products/detail/kemet/C0603C104K5RAC7867/1465623?utm_adgroup=Ceramic%20Capacitors&utm_source=google&utm_medium=cpc&utm_campaign=Shopping_Product_Capacitors_NEW&utm_term=&utm_content=Ceramic%20Capacitors" (id 5) (at 115.57 90.17 0)
+    (property "Stock" "https://www.digikey.com/en/products/detail/kemet/C0603C104K5RAC3190/12701955?utm_adgroup=Capacitors&utm_source=google&utm_medium=cpc&utm_campaign=Shopping_Supplier_KEMET&utm_term=&utm_content=Capacitors" (id 5) (at 115.57 90.17 0)
       (effects (font (size 1.27 1.27)) hide)
     )

Commit message: changed LED resistor value
Parts:
- R7: value 1k -> 10k; MPN RES SMD 1K OHM 1% 1/8W 0603 -> RES 10K OHM 1% 1/10W 0603; Stock https://www.digikey.com/en/products/detail/stackpole-electr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 -> https://www.digikey.com/en/products/detail/vishay-dale/CRCW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
Changed lines of the file:
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@@
       (effects (font (size 1.27 1.27)) (justify left))
     )
-    (property "Value" "1k" (id 1) (at 147.32 55.8799 0)
+    (property "Value" "10k" (id 1) (at 147.32 55.8799 0)
       (effects (font (size 1.27 1.27)) (justify left))
     )
@@
       (effects (font (size 1.27 1.27)) hide)
     )
-    (property "MPN" "RES SMD 1K OHM 1% 1/8W 0603" (id 4) (at 144.78 54.61 0)
+    (property "MPN" "RES 10K OHM 1% 1/10W 0603" (id 4) (at 144.78 54.61 0)
       (effects (font (size 1.27 1.27)) hide)
     )
-    (property "Stock" "https://www.digikey.com/en/products/detail/stackpole-electronics-inc/RNCP0603FTD1K00/2240106" (id 5) (at 144.78 54.61 0)
+    (property "Stock" "https://www.digikey.com/en/products/detail/vishay-dale/CRCW060310K0FKECC/12744930?utm_adgroup=Resistors&utm_source=google&utm_medium=cpc&utm_campaign=Shopping_Supplier_Vishay&utm_term=&utm_content=Resistors" (id 5) (at 144.78 54.61 0)
       (effects (font (size 1.27 1.27)) hide)
     )
