File: Hardware/System/backpackbuddy_system/power.kicad_sch (KiCad schematic)
At the start: 35 parts, among them J11 Battery, Q3 SIHF9Z24STRR-GE3, U2 SI-8050Y, U3 LM3940

Commit message: pp: flipped Q3 pins, changed values for D3 and D5 and updated datasheets; also fixed solder jump short pp such that its fused
Parts:
- D3: value 10V -> 20V; MPN NZH10C -> NZH20C,115; Stock https://www.digikey.com/en/products/detail/nexperia-usa-inc/NZH10C-115/2296361?utm_adgroup=Semiconductor%20Modules&utm_source=google&utm_medium=cpc&utm_campaign=Dynamic%20Search_EN_Product&utm_term=&utm_content=Semiconductor%20Modules -> https://www.digikey.com/en/products/detail/nexperia-usa-inc/NZH20C-115/2296368
- D5: value 18V -> 27V; MPN NZH18C -> DFLZ27-TP; Stock https://www.digikey.com/en/products/detail/nexperia-usa-inc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 -> https://www.digikey.com/en/products/detail/micro-commercial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
Connections:
- net 18V PROTECTED: now also Q3.2 (D); no longer Q3.3 (S)
- net at F2.1, J11.2 (Pin_2): no longer JP1.1 (A)
- net at D2.2 (A), F2.2, TP1.1: now also JP1.1 (A), Q3.3 (S); no longer Q3.2 (D)
Other:
- moved on the sheet: F2, Q3
Changed lines of the file:
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@@
   (junction (at 96.52 97.79) (diameter 0) (color 0 0 0 0)
   )
+  (junction (at 67.31 48.26) (diameter 0) (color 0 0 0 0)
+  )
   (junction (at 82.55 48.26) (diameter 0) (color 0 0 0 0)
   )
@@
   (junction (at 135.89 82.55) (diameter 0) (color 0 0 0 0)
   )
-  (junction (at 52.07 48.26) (diameter 0) (color 0 0 0 0)
-  )
   (junction (at 147.32 139.7) (diameter 0) (color 0 0 0 0)
   )
@@
     (stroke (width 0) (type default) (color 0 0 0 0))
   )
+  (wire (pts (xy 67.31 33.02) (xy 67.31 48.26))
+    (stroke (width 0) (type default) (color 0 0 0 0))
+  )
   (wire (pts (xy 259.08 44.45) (xy 264.16 44.45))
     (stroke (width 0) (type default) (color 0 0 0 0))
@@
     (stroke (width 0) (type default) (color 0 0 0 0))
   )
-  (wire (pts (xy 52.07 33.02) (xy 52.07 48.26))
-    (stroke (width 0) (type default) (color 0 0 0 0))
-  )
   (wire (pts (xy 135.89 93.98) (xy 135.89 97.79))
     (stroke (width 0) (type default) (color 0 0 0 0))
@@
     (stroke (width 0) (type default) (color 0 0 0 0))
   )
+  (wire (pts (xy 119.38 33.02) (xy 67.31 33.02))
+    (stroke (width 0) (type default) (color 0 0 0 0))
+  )
   (wire (pts (xy 96.52 97.79) (xy 96.52 100.33))
     (stroke (width 0) (type default) (color 0 0 0 0))
@@
     (stroke (width 0) (type default) (color 0 0 0 0))
   )
+  (wire (pts (xy 57.15 48.26) (xy 67.31 48.26))
+    (stroke (width 0) (type default) (color 0 0 0 0))
+  )
   (wire (pts (xy 96.52 48.26) (xy 102.87 48.26))
     (stroke (width 0) (type default) (color 0 0 0 0))
@@
     (stroke (width 0) (type default) (color 0 0 0 0))
   )
-  (wire (pts (xy 119.38 33.02) (xy 52.07 33.02))
-    (stroke (width 0) (type default) (color 0 0 0 0))
-  )
   (wire (pts (xy 144.78 48.26) (xy 144.78 50.8))
     (stroke (width 0) (type default) (color 0 0 0 0))
@@
     (stroke (width 0) (type default) (color 0 0 0 0))
   )
+  (wire (pts (xy 67.31 48.26) (xy 82.55 48.26))
+    (stroke (width 0) (type default) (color 0 0 0 0))
+  )
   (wire (pts (xy 212.09 55.88) (xy 212.09 58.42))
     (stroke (width 0) (type default) (color 0 0 0 0))
@@
     (stroke (width 0) (type default) (color 0 0 0 0))
   )
-  (wire (pts (xy 52.07 48.26) (xy 64.77 48.26))
-    (stroke (width 0) (type default) (color 0 0 0 0))
-  )
   (wire (pts (xy 46.99 130.81) (xy 59.69 130.81))
     (stroke (width 0) (type default) (color 0 0 0 0))
@@
     (stroke (width 0) (type default) (color 0 0 0 0))
   )
-  (wire (pts (xy 72.39 48.26) (xy 82.55 48.26))
-    (stroke (width 0) (type default) (color 0 0 0 0))
-  )
   (wire (pts (xy 93.98 160.02) (xy 93.98 163.83))
     (stroke (width 0) (type default) (color 0 0 0 0))
@@
     (stroke (width 0) (type default) (color 0 0 0 0))
   )
-  (wire (pts (xy 40.64 48.26) (xy 52.07 48.26))
+  (wire (pts (xy 40.64 48.26) (xy 49.53 48.26))
     (stroke (width 0) (type default) (color 0 0 0 0))
   )
@@
       (effects (font (size 1.27 1.27)) (justify left))
     )
-    (property "Value" "10V" (id 1) (at 118.11 55.8799 90)
+    (property "Value" "20V" (id 1) (at 118.11 55.8799 90)
       (effects (font (size 1.27 1.27)) (justify left))
     )
@@
       (effects (font (size 1.27 1.27)) hide)
     )
-    (property "Datasheet" "https://assets.nexperia.com/documents/data-sheet/NZH_SER.pdf" (id 3) (at 115.57 54.61 0)
-      (effects (font (size 1.27 1.27)) hide)
-    )
-    (property "MPN" "NZH10C" (id 4) (at 115.57 54.61 0)
-      (effects (font (size 1.27 1.27)) hide)
-    )
-    (property "Stock" "https://www.digikey.com/en/products/detail/nexperia-usa-inc/NZH10C-115/2296361?utm_adgroup=Semiconductor%20Modules&utm_source=google&utm_medium=cpc&utm_campaign=Dynamic%20Search_EN_Product&utm_term=&utm_content=Semiconductor%20Modules" (id 5) (at 115.57 54.61 0)
+    (property "Datasheet" "https://rocelec.widen.net/view/pdf/v8ln07ctm8/NEXP-S-A0002880914-1.pdf?t.download=true&u=5oefqw" (id 3) (at 115.57 54.61 0)
+      (effects (font (size 1.27 1.27)) hide)
+    )
+    (property "MPN" "NZH20C,115" (id 4) (at 115.57 54.61 0)
+      (effects (font (size 1.27 1.27)) hide)
+    )
+    (property "Stock" "https://www.digikey.com/en/products/detail/nexperia-usa-inc/NZH20C-115/2296368" (id 5) (at 115.57 54.61 0)
       (effects (font (size 1.27 1.27)) hide)
     )
@@
       (effects (font (size 1.27 1.27)) (justify left))
     )
-    (property "Value" "18V" (id 1) (at 138.43 66.0399 90)
+    (property "Value" "27V" (id 1) (at 138.43 66.0399 90)
       (effects (font (size 1.27 1.27)) (justify left))
     )
@@
       (effects (font (size 1.27 1.27)) hide)
     )
-    (property "Datasheet" "https://assets.nexperia.com/documents/data-sheet/NZH_SER.pdf" (id 3) (at 135.89 64.77 0)
-      (effects (font (size 1.27 1.27)) hide)
-    )
-    (property "MPN" "NZH18C" (id 4) (at 135.89 64.77 0)
-      (effects (font (size 1.27 1.27)) hide)
-    )
-    (property "Stock" "https://www.digikey.com/en/products/detail/nexperia-usa-inc/NZH18C-115/2296367" (id 5) (at 135.89 64.77 0)
+    (property "Datasheet" "https://www.mccsemi.com/pdf/Products/DFLZ5V1~DFLZ100(SOD-123FL).pdf" (id 3) (at 135.89 64.77 0)
+      (effects (font (size 1.27 1.27)) hide)
+    )
+    (property "MPN" "DFLZ27-TP" (id 4) (at 135.89 64.77 0)
+      (effects (font (size 1.27 1.27)) hide)
+    )
+    (property "Stock" "https://www.digikey.com/en/products/detail/micro-commercial-co/DFLZ27-TP/2512782" (id 5) (at 135.89 64.77 0)
       (effects (font (size 1.27 1.27)) hide)
     )
@@
     (pin "2")
   )
-  (symbol (lib_id "Device:Q_PMOS_GDS") (at 107.95 50.8 90) (unit 1)
+  (symbol (lib_id "Device:Q_PMOS_GDS") (at 107.95 50.8 270) (mirror x) (unit 1)
     (in_bom yes) (on_board yes) (fields_autoplaced)
     (property "Reference" "Q3" (id 0) (at 107.95 40.64 90))
     (property "Value" "SIHF9Z24STRR-GE3" (id 1) (at 107.95 43.18 90))
-    (property "Footprint" "Package_TO_SOT_SMD:TO-263-2" (id 2) (at 105.41 45.72 0)
+    (property "Footprint" "Package_TO_SOT_SMD:TO-263-2" (id 2) (at 110.49 45.72 0)
       (effects (font (size 1.27 1.27)) hide)
     )
@@
     (pin "2")
   )
-  (symbol (lib_id "Device:Fuse") (at 68.58 48.26 90) (unit 1)
-    (in_bom yes) (on_board yes) (fields_autoplaced)
-    (property "Reference" "F2" (id 0) (at 68.58 41.91 90))
-    (property "Value" "4A" (id 1) (at 68.58 44.45 90))
-    (property "Footprint" "Fuse:Fuse_0603_1608Metric_Pad1.05x0.95mm_HandSolder" (id 2) (at 68.58 50.038 90)
-      (effects (font (size 1.27 1.27)) hide)
-    )
-    (property "Datasheet" "https://www.mouser.com/datasheet/2/54/Bourns_SF_0603SPA_R_datasheet-2935204.pdf" (id 3) (at 68.58 48.26 0)
-      (effects (font (size 1.27 1.27)) hide)
-    )
-    (property "MPN" "SF-0603SPA500R-2" (id 4) (at 68.58 48.26 0)
-      (effects (font (size 1.27 1.27)) hide)
-    )
-    (property "Stock" "https://www.mouser.com/ProductDetail/Bourns/SF-0603SPA500R-2?qs=sGAEpiMZZMsIz3CjQ1xegZx2pdJYlyprauhgMChWNHkdzemHf%2F5IKw%3D%3D" (id 5) (at 68.58 48.26 0)
-      (effects (font (size 1.27 1.27)) hide)
-    )
+  (symbol (lib_id "Device:Fuse") (at 53.34 48.26 90) (unit 1)
+    (in_bom yes) (on_board yes) (fields_autoplaced)
+    (property "Reference" "F2" (id 0) (at 53.34 41.91 90))
+    (property "Value" "4A" (id 1) (at 53.34 44.45 90))
+    (property "Footprint" "Fuse:Fuse_0603_1608Metric_Pad1.05x0.95mm_HandSolder" (id 2) (at 53.34 50.038 90)
+      (effects (font (size 1.27 1.27)) hide)
+    )
+    (property "Datasheet" "https://www.mouser.com/datasheet/2/54/Bourns_SF_0603SPA_R_datasheet-2935204.pdf" (id 3) (at 53.34 48.26 0)
+      (effects (font (size 1.27 1.27)) hide)
+    )
+    (property "MPN" "SF-0603SPA500R-2" (id 4) (at 53.34 48.26 0)
+      (effects (font (size 1.27 1.27)) hide)
+    )
+    (property "Stock" "https://www.mouser.com/ProductDetail/Bourns/SF-0603SPA500R-2?qs=sGAEpiMZZMsIz3CjQ1xegZx2pdJYlyprauhgMChWNHkdzemHf%2F5IKw%3D%3D" (id 5) (at 53.34 48.26 0)
+      (effects (font (size 1.27 1.27)) hide)
+    )
