File: Hardware/System/backpackbuddy_system/power.kicad_sch (KiCad schematic)
At the start: 35 parts, among them J11 Battery, Q3 SIHF9Z24STRR-GE3, U2 SI-8050Y, U3 LM3940

Commit message: pp short
Parts:
- D6: value Red -> Vin
- D7: value Red -> 5V
- D8: value Red -> 3v3
Changed lines of the file:
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@@
       (effects (font (size 1.27 1.27)) (justify right))
     )
-    (property "Value" "Red" (id 1) (at 148.59 67.6274 90)
+    (property "Value" "Vin" (id 1) (at 148.59 67.6274 90)
       (effects (font (size 1.27 1.27)) (justify right))
     )
@@
       (effects (font (size 1.27 1.27)) (justify right))
     )
-    (property "Value" "Red" (id 1) (at 260.35 63.8174 90)
+    (property "Value" "3v3" (id 1) (at 260.35 63.8174 90)
       (effects (font (size 1.27 1.27)) (justify right))
     )
@@
       (effects (font (size 1.27 1.27)) (justify right))
     )
-    (property "Value" "Red" (id 1) (at 151.13 159.0674 90)
-      (effects (font (size 1.27 1.27)) (justify right))
-    )
+    (property "Value" "5V" (id 1) (at 151.13 159.0674 90)
+      (effects (font (size 1.27 1.27)) (justify right))
+    )
