File: Hardware/System/backpackbuddy_system/backpackbuddy_system.kicad_pcb (KiCad board)
At the start: 2 copper layers, 65 x 56 mm, 87 parts, among them J1 PIR, J10 USB_B_Micro, J11 Battery, J12 ICSP, J2 Ultrasonic 2, J3 Ultrasonic 1, J4 Left Vibration 1, J5 Left Vibration 2, J6 RPi_GPIO, J7 ESP8266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

Commit message: version 3 fixed some silkscreen
Parts:
- D10: value Green -> DB1
- D11: value Yellow -> DB2
- D12: value Amber -> DB3
- D6: value Red -> Vin
- D7: value Red -> 5V
- D8: value Red -> 3v3
- J4: value Left Vibration 1 -> Left Vibes
- J8: value Right Vibration 1 -> Right Vibes
- SW1: value ESP8266 RESET -> ESP RESET
- TP1: value 9V Unprotected -> Vin_U
- TP3: value Protected 9V -> Vin_P
Routing:
- net Net-(C12-Pad2): track 32.9 -> 28.5 mm
- net GND: track 295.1 -> 293.5 mm, vias 26 -> 25
- net /ESP RESET: track 19.0 -> 18.4 mm
Other:
- board text added: "Backpack Buddy Jeric Emily Rahul SP2023 V3"
- board text removed: "Backpack Buddy Jeric Emily Rahul SP2023"
Changed lines of the file:
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@@
       (effects (font (size 1 1) (thickness 0.15)))
     )
-    (fp_text value "Red" (at -0.4318 1.4732) (layer "F.SilkS")
+    (fp_text value "5V" (at -0.4318 1.4732) (layer "F.SilkS")
       (effects (font (size 1 1) (thickness 0.15)))
     )
@@
       (effects (font (size 1 1) (thickness 0.15)))
     )
-    (fp_text value "Left Vibration 1" (at 2.159 -2.5908) (layer "F.SilkS")
+    (fp_text value "Left Vibes" (at 2.159 -2.5908) (layer "F.SilkS")
       (effects (font (size 1 1) (thickness 0.15)))
     )
@@
       (effects (font (size 1 1) (thickness 0.15)))
     )
-    (fp_text value "Red" (at -3.175 -0.127) (layer "F.SilkS")
+    (fp_text value "Vin" (at -3.175 -0.127) (layer "F.SilkS")
       (effects (font (size 0.8 0.8) (thickness 0.15)))
     )
@@
       (effects (font (size 1 1) (thickness 0.15)))
     )
-    (fp_text value "Red" (at -0.381 1.651) (layer "F.SilkS")
+    (fp_text value "3v3" (at -0.381 1.651) (layer "F.SilkS")
       (effects (font (size 1 1) (thickness 0.15)))
     )
@@
       (effects (font (size 1 1) (thickness 0.15)))
     )
-    (fp_text value "Yellow" (at -2.286 -0.254 180) (layer "F.SilkS")
+    (fp_text value "DB2" (at -2.286 -0.254 180) (layer "F.SilkS")
       (effects (font (size 0.7 0.7) (thickness 0.15)))
     )
@@
     (property "Stock" "https://www.digikey.com/en/products/detail/kyocera-avx/08053D106KAT4A/12153448?utm_adgroup=Capacitors&utm_source=google&utm_medium=cpc&utm_campaign=Shopping_Supplier_AVX%20Corporation&utm_term=&utm_content=Capacitors")
     (attr smd)
-    (fp_text reference "C16" (at 0 -1.68) (layer "F.SilkS")
+    (fp_text reference "C16" (at -2.4625 -0.25 90) (layer "F.SilkS")
       (effects (font (size 1 1) (thickness 0.15)))
     )
@@
       (effects (font (size 1 1) (thickness 0.15)))
     )
-    (fp_text value "ESP8266 RESET" (at 1.016 -3.937 unlocked) (layer "F.SilkS")
+    (fp_text value "ESP RESET" (at 1.016 -3.937 unlocked) (layer "F.SilkS")
       (effects (font (size 1 1) (thickness 0.15)))
     )
@@
       (effects (font (size 1 1) (thickness 0.15)))
     )
-    (fp_text value "Right Vibration 1" (at 2.286 7.366) (layer "F.SilkS")
+    (fp_text value "Right Vibes" (at 2.286 7.366) (layer "F.SilkS")
       (effects (font (size 1 1) (thickness 0.15)))
     )
@@
       (effects (font (size 1 1) (thickness 0.15)))
     )
-    (fp_text value "9V Unprotected" (at -0.0508 -1.4986) (layer "F.SilkS")
+    (fp_text value "Vin_U" (at -0.0508 -1.4986) (layer "F.SilkS")
       (effects (font (size 0.7 0.7) (thickness 0.15)))
     )
@@
       (effects (font (size 1 1) (thickness 0.15)))
     )
-    (fp_text value "Green" (at -2.286 -0.381 180) (layer "F.SilkS")
+    (fp_text value "DB1" (at -2.286 -0.381 180) (layer "F.SilkS")
       (effects (font (size 0.7 0.7) (thickness 0.15)))
     )
@@
       (effects (font (size 1 1) (thickness 0.15)))
     )
-    (fp_text value "Protected 9V" (at 0.0254 -1.2954) (layer "F.SilkS")
+    (fp_text value "Vin_P" (at 0.0254 -1.2954) (layer "F.SilkS")
       (effects (font (size 0.7 0.7) (thickness 0.15)))
     )
@@
       (effects (font (size 1 1) (thickness 0.15)))
     )
-    (fp_text value "Amber" (at -2.3114 -0.0508 180) (layer "F.SilkS")
+    (fp_text value "DB3" (at -2.3114 -0.0508 180) (layer "F.SilkS")
       (effects (font (size 0.7 0.7) (thickness 0.15)))
     )
@@
     (property "Stock" "https://www.digikey.com/en/products/detail/bel-fuse-inc/0686F0500-01/7427694")
     (attr smd)
-    (fp_text reference "F1" (at 2.3114 0.0508 90) (layer "F.SilkS")
+    (fp_text reference "F1" (at 2.332 0.262 90) (layer "F.SilkS")
       (effects (font (size 1 1) (thickness 0.15)))
     )
@@
   (gr_line (start 176.036937 62.995948) (end 176.009999 113.03) (layer "Edge.Cuts") (width 0.1))
   (gr_arc (start 155.01 97) (mid 156.01 96) (end 157.01 97) (layer "Edge.Cuts") (width 0.1))
-  (gr_text "Backpack Buddy\nJeric\nEmily\nRahul\nSP2023" (at 145.923 102.616) (layer "F.SilkS")
+  (gr_text "Backpack Buddy\nJeric\nEmily\nRahul\nSP2023\nV3" (at 145.923 104.1) (layer "F.SilkS")
     (effects (font (size 1 1) (thickness 0.15)))
   )
@@
   (segment (start 121.92 67.945) (end 121.115 67.945) (width 0.25) (layer "F.Cu") (net 1))
   (segment (start 137.287 94.869) (end 136.616 95.54) (width 1) (layer "F.Cu") (net 1))
-  (segment (start 156.9935 93.472) (end 157.226 93.2395) (width 0.25) (layer "F.Cu") (net 1))
   (segment (start 137.414 102.7325) (end 137.541 102.6055) (width 0.25) (layer "F.Cu") (net 1))
   (segment (start 130.556 110.5115) (end 130.5775 110.49) (width 1) (layer "F.Cu") (net 1))
@@
   (segment (start 124.877 95.54) (end 124.2695 94.9325) (width 0.25) (layer "F.Cu") (net 1))
   (segment (start 166.25 113.2048) (end 166.8372 113.792) (width 0.25) (layer "F.Cu") (net 1))
-  (segment (start 128.778 83.439) (end 127.7874 83.439) (width 0.25) (layer "F.Cu") (net 1))
   (segment (start 128.6073 67.6331) (end 128.0808 68.1596) (width 1) (layer "F.Cu") (net 1))
   (segment (start 136.525 81.647) (end 136.525 83.4644) (width 0.25) (layer "F.Cu") (net 1))
@@
   (segment (start 116.84 71.12) (end 113.284 71.12) (width 1) (layer "F.Cu") (net 1))
   (segment (start 127.279 78.08) (end 128.64 78.08) (width 1) (layer "F.Cu") (net 1))
-  (segment (start 128.5475 83.6695) (end 128.778 83.439) (width 0.25) (layer "F.Cu") (net 1))
   (segment (start 138.2382 108.2434) (end 137.3378 109.1438) (width 0.25) (layer "F.Cu") (net 1))
   (segment (start 128.0808 68.1596) (end 128.0808 68.834) (width 1) (layer "F.Cu") (net 1))
@@
   (via (at 128.0054 95.54) (size 0.6) (drill 0.4) (layers "F.Cu" "B.Cu") (net 1))
   (via (at 127.279 78.08) (size 0.6) (drill 0.4) (layers "F.Cu" "B.Cu") (net 1))
-  (via (at 119.507 71.1708) (size 1.2) (drill 0.8) (layers "F.Cu" "B.Cu") (free) (net 1))
   (via (at 131.9424 95.54) (size 0.6) (drill 0.4) (layers "F.Cu" "B.Cu") (net 1))
   (via (at 129.7432 103.5558) (size 0.6) (drill 0.4) (layers "F.Cu" "B.Cu") (free) (net 1))
@@
   (segment (start 147.32 110.49) (end 147.325 110.495) (width 0.25) (layer "F.Cu") (net 6))
   (segment (start 147.325 110.495) (end 147.325 113.792) (width 1) (layer "F.Cu") (net 6))
-  (segment (start 164.465 113.6242) (end 164.2972 113.792) (width 1) (layer "F.Cu") (net 6))
   (segment (start 128.524 113.538) (end 128.524 111.125) (width 1) (layer "F.Cu") (net 6))
   (segment (start 164.525 105.15) (end 163.79 105.885) (width 0.25) (layer "F.Cu") (net 6))
@@
   (via (at 151.892 78.74) (size 0.6) (drill 0.4) (layers "F.Cu" "B.Cu") (net 7))
   (segment (start 144.647 73.908) (end 148.209 77.47) (width 0.5) (layer "B.Cu") (net 7))
-  (segment (start 159.639 77.0675) (end 159.639 77.343) (width 0.25) (layer "B.Cu") (net 7))
   (segment (start 159.639 77.5785) (end 159.5305 77.47) (width 0.5) (layer "B.Cu") (net 7))
   (segment (start 159.639 77.343) (end 159.639 77.47) (width 0.25) (layer "B.Cu") (net 7))
@@
   (segment (start 157.5 73.05) (end 158.5 72.05) (width 1) (layer "F.Cu") (net 13))
   (segment (start 164.93 78.15) (end 165.735 78.955) (width 1) (layer "F.Cu") (net 13))
-  (segment (start 157.5 76.835) (end 157.5 80.284) (width 1) (layer "F.Cu") (net 13))
-  (segment (start 157.5 80.284) (end 158.171 80.955) (width 1) (layer "F.Cu") (net 13))
   (segment (start 157.5 76.835) (end 157.5 73.05) (width 1) (layer "F.Cu") (net 13))
   (segment (start 156.718 73.533) (end 155.194 73.533) (width 1) (layer "F.Cu") (net 13))
@@
   (segment (start 162 95.25) (end 162 104.3) (width 0.25) (layer "B.Cu") (net 57))
   (segment (start 124.714 87.285) (end 126.31 87.285) (width 0.25) (layer "F.Cu") (net 58))
-  (segment (start 120.885 87.285) (end 120.65 87.05) (width 0.25) (layer "F.Cu") (net 58))
   (segment (start 126.9473 85.1916) (end 126.9473 86.6477) (width 0.25) (layer "F.Cu") (net 58))
   (segment (start 126.9473 86.6477) (end 126.31 87.285) (width 0.25) (layer "F.Cu") (net 58))
@@
   (via (at 124.714 87.285) (size 0.6) (drill 0.4) (layers "F.Cu" "B.Cu") (net 58))
   (segment (start 124.714 87.285) (end 120.885 87.285) (width 0.25) (layer "B.Cu") (net 58))
-  (segment (start 120.885 87.285) (end 120.65 87.05) (width 0.25) (layer "B.Cu") (net 58))
   (segment (start 120.039 73.726) (end 113.35 73.726) (width 0.75) (layer "B.Cu") (net 59))
   (segment (start 113.35 73.726) (end 113.284 73.66) (width 0.25) (layer "B.Cu") (net 59))
@@
   (segment (start 127.439698 67.749698) (end 124.46 64.77) (width 0.25) (layer "B.Cu") (net 78))
   (segment (start 131.445 70.229604) (end 128.965094 67.749698) (width 0.25) (layer "B.Cu") (net 78))
-  (segment (start 144.8435 100.1395) (end 144.78 100.203) (width 0.25) (layer "F.Cu") (net 80))
   (segment (start 144.8435 100.1395) (end 145.542 99.441) (width 0.25) (layer "F.Cu") (net 80))
   (segment (start 145.542 99.441) (end 145.542 94.361) (width 0.25) (layer "F.Cu") (net 80))

Commit message: pp short
Routing:
- net GND: track 293.5 -> 285.2 mm
- net +5V: track 75.4 -> 71.3 mm
- net /RESET: track 78.1 -> 77.1 mm
- net /Power/18V PROTECTED: track 81.3 -> 80.3 mm
- net Net-(C12-Pad2): track 28.5 -> 29.1 mm
- net Net-(C10-Pad1): track 15.4 -> 14.9 mm
